File: superlna.sch (EAGLE design)
At the start: 7 parts, among them X1 SMA-142-0701-801/806, X2 SMA-142-0701-801/806

Commit message: V1.0
Parts:
- removed FILTER: BANDPASS, custom:BANDPASS
- removed PSA4-5043+: AMP, custom:AMP
- added C2, C3: (no value), rcl:C-USC0402
- added D1: BAV199, diode:BAV199
- added F1: BANDPASS, custom:BANDPASS
- added J2, L2: (no value), rcl:R-EU_R0805
- added POWER: (no value), microusb:USB""
- added U1: BIASTEE, minicircuits:BIASTEE
- added U2: AMP, custom:AMP
- J1: device rcl:R-US_R0805 -> rcl:R-EU_R0805
Connections:
- removed net N$1: FILTER.RFIN, L1.1, X1.1
- removed net N$3: C1.2, FILTER.RFOUT
- new net BIASPOWER: C1.1, J2.2, U1.3
- new net N$4: C3.1, J1.1, J2.1, L2.1, POWER.VBUS
- new net N$6: F1.RFIN, U1.2
- new net RFIN: C2.2, D1.AC, L1.1, X1.1
- new net RFOUT: F1.RFOUT, L2.2, X2.1
- net GND: now also C1.2, C3.2, D1.A, D1.C, F1.GND, POWER.GND, U1.GND, U2.GND; no longer FILTER.GND, PSA4-5043+.GND
- net N$2: now also C2.1, U2.RFIN; no longer C1.1, PSA4-5043+.RFIN
- net N$5: now also U1.1, U2.RF/DC-OUT; no longer J1.1, PSA4-5043+.RF/DC-OUT, X2.1
Other:
- moved on the sheet: C1, L1, X2

Commit message: changes to V1
Parts:
- removed U2: AMP, custom:AMP
- added U$1: AMP, minicircuits:AMP
Connections:
- net GND: now also U$1.GND; no longer U2.GND
- net N$2: now also U$1.RFIN; no longer U2.RFIN
- net N$5: now also U$1.RF/DC-OUT; no longer U2.RF/DC-OUT
Changed lines of the file:
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@@
 <part name="SUPPLY5" library="supply2" deviceset="GND" device=""/>
 <part name="C2" library="rcl" deviceset="C-US" device="C0402"/>
-<part name="U2" library="custom" deviceset="AMP" device=""/>
 <part name="U1" library="minicircuits" deviceset="BIASTEE" device=""/>
 <part name="SUPPLY7" library="supply2" deviceset="GND" device=""/>
+<part name="U$1" library="minicircuits" deviceset="AMP" device=""/>
 </parts>
 <sheets>
@@
 <instance part="SUPPLY5" gate="GND" x="53.34" y="50.8"/>
 <instance part="C2" gate="G$1" x="-22.86" y="2.54" rot="R270"/>
-<instance part="U2" gate="G$1" x="17.78" y="2.54"/>
 <instance part="U1" gate="G$1" x="73.66" y="2.54"/>
 <instance part="SUPPLY7" gate="GND" x="73.66" y="-20.32"/>
+<instance part="U$1" gate="G$1" x="17.78" y="2.54"/>
 </instances>
 <busses>
@@
 <wire x1="17.78" y1="-17.78" x2="17.78" y2="-22.86" width="0.1524" layer="91"/>
 <pinref part="SUPPLY3" gate="GND" pin="GND"/>
-<pinref part="U2" gate="G$1" pin="GND"/>
+<pinref part="U$1" gate="G$1" pin="GND"/>
 </segment>
 <segment>
@@
 <segment>
 <wire x1="55.88" y1="2.54" x2="48.26" y2="2.54" width="0.1524" layer="91"/>
-<pinref part="U2" gate="G$1" pin="RF/DC-OUT"/>
 <pinref part="U1" gate="G$1" pin="1"/>
+<pinref part="U$1" gate="G$1" pin="RF/DC-OUT"/>
 </segment>
 </net>
@@
 <segment>
 <pinref part="C2" gate="G$1" pin="1"/>
-<pinref part="U2" gate="G$1" pin="RFIN"/>
+<pinref part="U$1" gate="G$1" pin="RFIN"/>
 <wire x1="-20.32" y1="2.54" x2="0" y2="2.54" width="0.1524" layer="91"/>
 </segment>

Commit message: V2
Parts:
- removed X2: SMA-142-0701-801/806, con-coax:SMA-142-0701-801/806
- added LED1: (no value), eagle-ltspice:LED_ESML0603
- added RFIN: SMA-142-0711-821/826, con-coax:SMA-142-0711-821/826
- X1: value SMA-142-0701-801/806 -> SMA-142-0711-821/826; device con-coax:SMA-142-0701-801/806 -> con-coax:SMA-142-0711-821/826
- renumbered U$1 to LNA
Connections:
- net N$6 renamed RFOUT1
- removed net N$4: C3.1, J1.1, J2.1, L2.1, POWER.VBUS
- new net PWRIN: C3.1, J1.1, J2.1, L2.1, LED1.A, POWER.VBUS
- net GND: now also LED1.C, RFIN.2; no longer X2.2
- net RFIN: now also RFIN.1; no longer X1.1
- net RFOUT: now also X1.1; no longer X2.1
Other:
- moved on the sheet: X1
Changed lines of the file:
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@@
 </classes>
 <parts>
-<part name="X1" library="con-coax" deviceset="SMA-" device="142-0701-801/806"/>
 <part name="L1" library="rcl" deviceset="R-EU_" device="R0805"/>
-<part name="X2" library="con-coax" deviceset="SMA-" device="142-0701-801/806"/>
 <part name="SUPPLY2" library="supply2" deviceset="GND" device=""/>
 <part name="SUPPLY3" library="supply2" deviceset="GND" device=""/>
@@
 <part name="U1" library="minicircuits" deviceset="BIASTEE" device=""/>
 <part name="SUPPLY7" library="supply2" deviceset="GND" device=""/>
-<part name="U$1" library="minicircuits" deviceset="AMP" device=""/>
+<part name="LNA" library="minicircuits" deviceset="AMP" device=""/>
+<part name="RFIN" library="con-coax" deviceset="SMA-" device="142-0711-821/826"/>
+<part name="X1" library="con-coax" deviceset="SMA-" device="142-0711-821/826"/>
+<part name="LED1" library="eagle-ltspice" deviceset="LED_E" device="SML0603"/>
+<part name="SUPPLY8" library="supply2" deviceset="GND" device=""/>
 </parts>
 <sheets>
@@
 </plain>
 <instances>
-<instance part="X1" gate="G1" x="-55.88" y="2.54"/>
 <instance part="L1" gate="G$1" x="-43.18" y="7.62" rot="R90"/>
-<instance part="X2" gate="G1" x="170.18" y="2.54" rot="R180"/>
 <instance part="SUPPLY2" gate="GND" x="-43.18" y="-15.24"/>
 <instance part="SUPPLY3" gate="GND" x="17.78" y="-25.4"/>
@@
 <instance part="U1" gate="G$1" x="73.66" y="2.54"/>
 <instance part="SUPPLY7" gate="GND" x="73.66" y="-20.32"/>
-<instance part="U$1" gate="G$1" x="17.78" y="2.54"/>
+<instance part="LNA" gate="G$1" x="17.78" y="2.54"/>
+<instance part="RFIN" gate="G1" x="-55.88" y="2.54"/>
+<instance part="X1" gate="G1" x="170.18" y="2.54" rot="R180"/>
+<instance part="LED1" gate="G$1" x="50.8" y="30.48"/>
+<instance part="SUPPLY8" gate="GND" x="50.8" y="20.32"/>
 </instances>
 <busses>
@@
 <wire x1="17.78" y1="-17.78" x2="17.78" y2="-22.86" width="0.1524" layer="91"/>
 <pinref part="SUPPLY3" gate="GND" pin="GND"/>
-<pinref part="U$1" gate="G$1" pin="GND"/>
+<pinref part="LNA" gate="G$1" pin="GND"/>
 </segment>
 <segment>
-<pinref part="X2" gate="G1" pin="2"/>
 <wire x1="167.64" y1="5.08" x2="149.86" y2="5.08" width="0.1524" layer="91"/>
 <wire x1="149.86" y1="5.08" x2="149.86" y2="-7.62" width="0.1524" layer="91"/>
 <pinref part="SUPPLY4" gate="GND" pin="GND"/>
+<pinref part="X1" gate="G1" pin="2"/>
 </segment>
 <segment>
@@
 </segment>
 <segment>
-<pinref part="X1" gate="G1" pin="2"/>
 <pinref part="D1" gate="G$1" pin="C"/>
 <wire x1="-53.34" y1="-7.62" x2="-53.34" y2="0" width="0.1524" layer="91"/>
@@
 <pinref part="SUPPLY2" gate="GND" pin="GND"/>
 <junction x="-43.18" y="-12.7"/>
+<pinref part="RFIN" gate="G1" pin="2"/>
 </segment>
 <segment>
@@
 <wire x1="73.66" y1="-17.78" x2="73.66" y2="-12.7" width="0.1524" layer="91"/>
 </segment>
+<segment>
+<pinref part="LED1" gate="G$1" pin="C"/>
+<pinref part="SUPPLY8" gate="GND" pin="GND"/>
+<wire x1="50.8" y1="22.86" x2="50.8" y2="25.4" width="0.1524" layer="91"/>
+</segment>
 </net>
 <net name="RFIN" class="0">
 <segment>
-<pinref part="X1" gate="G1" pin="1"/>
 <wire x1="-53.34" y1="2.54" x2="-43.18" y2="2.54" width="0.1524" layer="91"/>
 <pinref part="L1" gate="G$1" pin="1"/>
@@
 <wire x1="-43.18" y1="-5.08" x2="-43.18" y2="2.54" width="0.1524" layer="91"/>
 <pinref part="C2" gate="G$1" pin="2"/>
+<pinref part="RFIN" gate="G1" pin="1"/>
 </segment>
 </net>
-<net name="N$4" class="0">
+<net name="PWRIN" class="0">
 <segment>
 <pinref part="POWER" gate="G$1" pin="VBUS"/>
@@
 <wire x1="66.04" y1="45.72" x2="66.04" y2="43.18" width="0.1524" layer="91"/>
 <pinref part="J1" gate="G$1" pin="1"/>
-<wire x1="15.24" y1="33.02" x2="73.66" y2="33.02" width="0.1524" layer="91"/>
+<wire x1="15.24" y1="33.02" x2="50.8" y2="33.02" width="0.1524" layer="91"/>
 <pinref part="L2" gate="G$1" pin="1"/>
+<wire x1="50.8" y1="33.02" x2="73.66" y2="33.02" width="0.1524" layer="91"/>
 <wire x1="139.7" y1="12.7" x2="139.7" y2="33.02" width="0.1524" layer="91"/>
 <wire x1="139.7" y1="33.02" x2="73.66" y2="33.02" width="0.1524" layer="91"/>
 <junction x="73.66" y="33.02"/>
 <pinref part="J2" gate="G$1" pin="1"/>
+<pinref part="LED1" gate="G$1" pin="A"/>
+<junction x="50.8" y="33.02"/>
 </segment>
 </net>
@@
 <wire x1="55.88" y1="2.54" x2="48.26" y2="2.54" width="0.1524" layer="91"/>
 <pinref part="U1" gate="G$1" pin="1"/>
-<pinref part="U$1" gate="G$1" pin="RF/DC-OUT"/>
+<pinref part="LNA" gate="G$1" pin="RF/DC-OUT"/>
 </segment>
 </net>
-<net name="N$6" class="0">
+<net name="RFOUT1" class="0">
 <segment>
 <wire x1="91.44" y1="2.54" x2="96.52" y2="2.54" width="0.1524" layer="91"/>
@@
 <net name="RFOUT" class="0">
 <segment>
-<pinref part="X2" gate="G1" pin="1"/>
 <pinref part="F1" gate="G$1" pin="RFOUT"/>
 <wire x1="167.64" y1="2.54" x2="139.7" y2="2.54" width="0.1524" layer="91"/>
@@
 <wire x1="139.7" y1="2.54" x2="132.08" y2="2.54" width="0.1524" layer="91"/>
 <junction x="139.7" y="2.54"/>
+<pinref part="X1" gate="G1" pin="1"/>
 </segment>
 </net>
@@
 <segment>
 <pinref part="C2" gate="G$1" pin="1"/>
-<pinref part="U$1" gate="G$1" pin="RFIN"/>
+<pinref part="LNA" gate="G$1" pin="RFIN"/>
 <wire x1="-20.32" y1="2.54" x2="0" y2="2.54" width="0.1524" layer="91"/>
 </segment>
